Commit message: Fix control issues found during inital testing.

File: tinykart_description/urdf/tinykart_robot.urdf (robot description, URDF)
Before this commit: robot tinykart, 10 links, 9 joints
Links:
- link left_front_wheel_rack: mass 0 -> 1.125
- link right_front_wheel: mass 0.1 -> 1.125
- link right_front_wheel_rack: mass 0 -> 1.125
