Commit message: being moving to ackermann

File: tinykart_description/urdf/tinykart.urdf (robot description, URDF)
Before this commit: robot tinykart, 15 links, 14 joints
Links:
- removed link camera_link
- removed link front_mast_pillar
- removed link left_mid_wheel
- removed link mid_mast_pillar
- removed link rear_mast_pillar
- removed link right_mid_wheel
- removed link top_mast_pillar
- added link left_front_wheel_rack, mass 2.25; visual cylinder length=0.1 radius=0.165
- added link right_front_wheel_rack, mass 2.25; visual cylinder length=0.1 radius=0.165
Joints:
- removed joint camera_link_to_base_link
- removed joint front_mast_pillar_to_base_link
- removed joint left_front_wheel_to_base_link
- removed joint left_mid_wheel_to_base_link
- removed joint mid_mast_pillar_to_base_link
- removed joint rear_mast_pillar_to_base_link
- removed joint right_front_wheel_to_base_link
- removed joint right_mid_wheel_to_base_link
- removed joint top_mast_pillar_to_base_link
- added joint left_front_wheel_rack_to_wheel: type continuous, parent left_front_wheel_rack, child left_front_wheel, origin xyz=0 -0.00001 0 rpy=0 0 0, axis 0 1 0
- added joint left_front_wheel_steer: type revolute, parent base_link, child left_front_wheel_rack, origin xyz=0.285 0.27 -0.0508 rpy=0 0 0, axis 0 0 1, limit lower=-0.6 upper=+0.6 effort=25 velocity=10.0
- added joint right_front_wheel_rack_to_wheel: type continuous, parent right_front_wheel_rack, child right_front_wheel, origin xyz=0 -0.00001 0 rpy=0 0 0, axis 0 1 0
- added joint right_front_wheel_steer: type revolute, parent base_link, child right_front_wheel_rack, origin xyz=0.285 -0.27 -0.0508 rpy=0 0 0, axis 0 0 1, limit lower=-0.6 upper=+0.6 effort=25 velocity=10.0

Commit message: mess with sim

File: tinykart_description/urdf/tinykart.urdf (robot description, URDF)
Before this commit: robot tinykart, 10 links, 9 joints
Links:
- link base_link: mass 28 -> 14; geometry collision box size=0.45 0.22 0.125; visual box size=0.45 0.22 0.125
- link laser_link: mass 1 -> 0
- link left_front_wheel: mass 2.25 -> 1.125; geometry collision cylinder length=0.1 radius=0.0825; visual cylinder length=0.1 radius=0.0825
- link left_front_wheel_rack: mass 2.25 -> 1.125; geometry visual cylinder length=0.1 radius=0.0825
- link left_rear_wheel: mass 2.25 -> 1.125; geometry collision cylinder length=0.1 radius=0.0825; visual cylinder length=0.1 radius=0.0825
- link right_front_wheel: mass 2.25 -> 1.125; geometry collision cylinder length=0.1 radius=0.0825; visual cylinder length=0.1 radius=0.0825
- link right_front_wheel_rack: mass 2.25 -> 1.125; geometry visual cylinder length=0.1 radius=0.0825
- link right_rear_wheel: mass 2.25 -> 1.125; geometry collision cylinder length=0.1 radius=0.0825; visual cylinder length=0.1 radius=0.0825
Joints:
- joint base_footprint_to_base_link: origin xyz=0 0 0.225 rpy=0 0 0 -> xyz=0 0 0.125 rpy=0 0 0
- joint left_front_wheel_steer: origin xyz=0.285 0.27 -0.0508 rpy=0 0 0 -> xyz= 0.1425 0.135 -0.0508 rpy=0 0 0
- joint left_rear_wheel_to_base_link: origin xyz=-0.285 0.27 -0.0508 rpy=0 0 0 -> xyz=-0.1425 0.135 -0.0508 rpy=0 0 0
- joint right_front_wheel_steer: origin xyz=0.285 -0.27 -0.0508 rpy=0 0 0 -> xyz=0.1425 -0.135 -0.0508 rpy=0 0 0
- joint right_rear_wheel_to_base_link: origin xyz=-0.285 -0.27 -0.0508 rpy=0 0 0 -> xyz=-0.1425 -0.135 -0.0508 rpy=0 0 0

Commit message: make like half of a urdf

File: tinykart_description/urdf/tinykart.urdf (robot description, URDF)
Before this commit: robot tinykart, 10 links, 9 joints
Links:
- link base_link: mass 14 -> 1; geometry collision box size=0.55245 0.19 0.02; visual box size=0.55245 0.19 0.02
- link left_front_wheel: mass 1.125 -> 0.1; geometry collision cylinder length=0.04 radius=0.05; visual cylinder length=0.04 radius=0.05
- link left_rear_wheel: mass 1.125 -> 0.1; geometry collision cylinder length=0.04 radius=0.05; visual cylinder length=0.04 radius=0.05
- link right_rear_wheel: mass 1.125 -> 0.1; geometry collision cylinder length=0.04 radius=0.05; visual cylinder length=0.04 radius=0.05
Joints:
- joint base_footprint_to_base_link: origin xyz=0 0 0.125 rpy=0 0 0 -> xyz=0 0 0.09525 rpy=0 0 0
- joint left_rear_wheel_to_base_link: origin xyz=-0.1425 0.135 -0.0508 rpy=0 0 0 -> xyz=-0.140575 0.095 -0.054 rpy=0 0 0
- joint right_rear_wheel_to_base_link: origin xyz=-0.1425 -0.135 -0.0508 rpy=0 0 0 -> xyz=-0.140575 -0.095 -0.054 rpy=0 0 0

File: tinykart_description/urdf/tinykart_robot.urdf (robot description, URDF)
Before this commit: robot tinykart, 15 links, 14 joints
Links:
- removed link camera_link
- removed link front_mast_pillar
- removed link left_mid_wheel
- removed link mid_mast_pillar
- removed link rear_mast_pillar
- removed link right_mid_wheel
- removed link top_mast_pillar
- added link left_front_wheel_rack, mass 0; visual box size=0.00001 0.0000001 0.000001
- added link right_front_wheel_rack, mass 0; visual box size=0.00001 0.0000001 0.000001
- link base_link: mass 28 -> 1; geometry collision box size=0.55245 0.19 0.02; visual box size=0.55245 0.19 0.02
- link laser_link: mass 1 -> 0
- link left_front_wheel: mass 2.25 -> 0.1; geometry collision cylinder length=0.04 radius=0.05; visual cylinder length=0.04 radius=0.05
- link left_rear_wheel: mass 2.25 -> 0.1; geometry collision cylinder length=0.04 radius=0.05; visual cylinder length=0.04 radius=0.05
- link right_front_wheel: mass 2.25 -> 0.1; geometry collision cylinder length=0.04 radius=0.05; visual cylinder length=0.04 radius=0.05
- link right_rear_wheel: mass 2.25 -> 0.1; geometry collision cylinder length=0.04 radius=0.05; visual cylinder length=0.04 radius=0.05
Joints:
- removed joint camera_link_to_base_link
- removed joint front_mast_pillar_to_base_link
- removed joint left_front_wheel_to_base_link
- removed joint left_mid_wheel_to_base_link
- removed joint mid_mast_pillar_to_base_link
- removed joint rear_mast_pillar_to_base_link
- removed joint right_front_wheel_to_base_link
- removed joint right_mid_wheel_to_base_link
- removed joint top_mast_pillar_to_base_link
- added joint left_front_wheel_rack_to_wheel: type continuous, parent left_front_wheel_rack, child left_front_wheel, origin xyz=0 -0.00001 0 rpy=0 0 0, axis 0 1 0
- added joint left_front_wheel_steer: type revolute, parent base_link, child left_front_wheel_rack, origin xyz=0.219075 0.095 -0.054 rpy=0 0 0, axis 0 0 1, limit lower=-0.3499 upper=+0.5236 effort=0.88269 velocity=3.0
- added joint right_front_wheel_rack_to_wheel: type continuous, parent right_front_wheel_rack, child right_front_wheel, origin xyz=0 -0.00001 0 rpy=0 0 0, axis 0 1 0
- added joint right_front_wheel_steer: type revolute, parent base_link, child right_front_wheel_rack, origin xyz= 0.219075 -0.095 -0.054 rpy=0 0 0, axis 0 0 1, limit lower=-0.3499 upper=+0.5236 effort=0.88269 velocity=3.0
- joint base_footprint_to_base_link: origin xyz=0.285 0 0.225 rpy=0 0 0 -> xyz=0 0 0.09525 rpy=0 0 0
- joint left_rear_wheel_to_base_link: origin xyz=-0.285 0.27 -0.0508 rpy=0 0 0 -> xyz=-0.140575 0.095 -0.054 rpy=0 0 0
- joint right_rear_wheel_to_base_link: origin xyz=-0.285 -0.27 -0.0508 rpy=0 0 0 -> xyz=-0.140575 -0.095 -0.054 rpy=0 0 0

Commit message: Everything but inertial values works

File: tinykart_description/urdf/tinykart.urdf (robot description, URDF)
Before this commit: robot tinykart, 10 links, 9 joints
Links:
- link left_front_wheel_rack: geometry visual box size=0.00001 0.0000001 0.000001
- link right_front_wheel: geometry collision cylinder length=0.04 radius=0.05; visual cylinder length=0.04 radius=0.05
- link right_front_wheel_rack: geometry visual box size=0.00001 0.0000001 0.000001
Joints:
- joint left_front_wheel_steer: limit lower=-0.6 upper=+0.6 effort=25 velocity=10.0 -> lower=-0.3499 upper=+0.5236 effort=0.88269 velocity=3.0; origin xyz= 0.1425 0.135 -0.0508 rpy=0 0 0 -> xyz=0.219075 0.095 -0.054 rpy=0 0 0
- joint right_front_wheel_steer: limit lower=-0.6 upper=+0.6 effort=25 velocity=10.0 -> lower=-0.3499 upper=+0.5236 effort=0.88269 velocity=3.0; origin xyz=0.1425 -0.135 -0.0508 rpy=0 0 0 -> xyz= 0.219075 -0.095 -0.054 rpy=0 0 0

Commit message: Urdf (#1)
* make like half of a urdf

* Everything but inertial values works

* Fix control issues found during inital testing.

File: tinykart_description/urdf/tinykart.urdf (robot description, URDF)
Before this commit: robot tinykart, 10 links, 9 joints
Links:
- link base_link: mass 14 -> 1; geometry collision box size=0.55245 0.19 0.02; visual box size=0.55245 0.19 0.02
- link left_front_wheel: mass 1.125 -> 0.1; geometry collision cylinder length=0.04 radius=0.05; visual cylinder length=0.04 radius=0.05
- link left_front_wheel_rack: geometry visual box size=0.00001 0.0000001 0.000001
- link left_rear_wheel: mass 1.125 -> 0.1; geometry collision cylinder length=0.04 radius=0.05; visual cylinder length=0.04 radius=0.05
- link right_front_wheel: geometry collision cylinder length=0.04 radius=0.05; visual cylinder length=0.04 radius=0.05
- link right_front_wheel_rack: geometry visual box size=0.00001 0.0000001 0.000001
- link right_rear_wheel: mass 1.125 -> 0.1; geometry collision cylinder length=0.04 radius=0.05; visual cylinder length=0.04 radius=0.05
Joints:
- joint base_footprint_to_base_link: origin xyz=0 0 0.125 rpy=0 0 0 -> xyz=0 0 0.09525 rpy=0 0 0
- joint left_front_wheel_steer: limit lower=-0.6 upper=+0.6 effort=25 velocity=10.0 -> lower=-0.3499 upper=+0.5236 effort=0.88269 velocity=3.0; origin xyz= 0.1425 0.135 -0.0508 rpy=0 0 0 -> xyz=0.219075 0.095 -0.054 rpy=0 0 0
- joint left_rear_wheel_to_base_link: origin xyz=-0.1425 0.135 -0.0508 rpy=0 0 0 -> xyz=-0.140575 0.095 -0.054 rpy=0 0 0
- joint right_front_wheel_steer: limit lower=-0.6 upper=+0.6 effort=25 velocity=10.0 -> lower=-0.3499 upper=+0.5236 effort=0.88269 velocity=3.0; origin xyz=0.1425 -0.135 -0.0508 rpy=0 0 0 -> xyz= 0.219075 -0.095 -0.054 rpy=0 0 0
- joint right_rear_wheel_to_base_link: origin xyz=-0.1425 -0.135 -0.0508 rpy=0 0 0 -> xyz=-0.140575 -0.095 -0.054 rpy=0 0 0

File: tinykart_description/urdf/tinykart_robot.urdf (robot description, URDF)
Before this commit: robot tinykart, 15 links, 14 joints
Links:
- removed link camera_link
- removed link front_mast_pillar
- removed link left_mid_wheel
- removed link mid_mast_pillar
- removed link rear_mast_pillar
- removed link right_mid_wheel
- removed link top_mast_pillar
- added link left_front_wheel_rack, mass 1.125; visual box size=0.00001 0.0000001 0.000001
- added link right_front_wheel_rack, mass 1.125; visual box size=0.00001 0.0000001 0.000001
- link base_link: mass 28 -> 1; geometry collision box size=0.55245 0.19 0.02; visual box size=0.55245 0.19 0.02
- link laser_link: mass 1 -> 0
- link left_front_wheel: mass 2.25 -> 0.1; geometry collision cylinder length=0.04 radius=0.05; visual cylinder length=0.04 radius=0.05
- link left_rear_wheel: mass 2.25 -> 0.1; geometry collision cylinder length=0.04 radius=0.05; visual cylinder length=0.04 radius=0.05
- link right_front_wheel: mass 2.25 -> 1.125; geometry collision cylinder length=0.04 radius=0.05; visual cylinder length=0.04 radius=0.05
- link right_rear_wheel: mass 2.25 -> 0.1; geometry collision cylinder length=0.04 radius=0.05; visual cylinder length=0.04 radius=0.05
Joints:
- removed joint camera_link_to_base_link
- removed joint front_mast_pillar_to_base_link
- removed joint left_front_wheel_to_base_link
- removed joint left_mid_wheel_to_base_link
- removed joint mid_mast_pillar_to_base_link
- removed joint rear_mast_pillar_to_base_link
- removed joint right_front_wheel_to_base_link
- removed joint right_mid_wheel_to_base_link
- removed joint top_mast_pillar_to_base_link
- added joint left_front_wheel_rack_to_wheel: type continuous, parent left_front_wheel_rack, child left_front_wheel, origin xyz=0 -0.00001 0 rpy=0 0 0, axis 0 1 0
- added joint left_front_wheel_steer: type revolute, parent base_link, child left_front_wheel_rack, origin xyz=0.219075 0.095 -0.054 rpy=0 0 0, axis 0 0 1, limit lower=-0.3499 upper=+0.5236 effort=0.88269 velocity=3.0
- added joint right_front_wheel_rack_to_wheel: type continuous, parent right_front_wheel_rack, child right_front_wheel, origin xyz=0 -0.00001 0 rpy=0 0 0, axis 0 1 0
- added joint right_front_wheel_steer: type revolute, parent base_link, child right_front_wheel_rack, origin xyz= 0.219075 -0.095 -0.054 rpy=0 0 0, axis 0 0 1, limit lower=-0.3499 upper=+0.5236 effort=0.88269 velocity=3.0
- joint base_footprint_to_base_link: origin xyz=0.285 0 0.225 rpy=0 0 0 -> xyz=0 0 0.09525 rpy=0 0 0
- joint left_rear_wheel_to_base_link: origin xyz=-0.285 0.27 -0.0508 rpy=0 0 0 -> xyz=-0.140575 0.095 -0.054 rpy=0 0 0
- joint right_rear_wheel_to_base_link: origin xyz=-0.285 -0.27 -0.0508 rpy=0 0 0 -> xyz=-0.140575 -0.095 -0.054 rpy=0 0 0

Commit message: wip

File: tinykart_description/urdf/tinykart.urdf (robot description, URDF)
Before this commit: robot tinykart, 10 links, 9 joints
Links:
- link base_link: mass 1 -> 2
- link imu_link: mass 1 -> 0
- link laser_link: geometry collision cylinder length=0.01 radius=0.00762; visual cylinder length=0.01 radius=0.00762
Joints:
- joint imu_link_to_base_link: origin xyz=-0.012 0 0.5588 rpy=0 0 0 -> xyz=-0.012 0 0.3 rpy=0 0 0
- joint laser_to_base_link: origin xyz=0.2722 0 0.3556 rpy=0 0 0 -> xyz=0.2722 0 0.2 rpy=0 0 0

File: tinykart_description/urdf/tinykart_robot.urdf (robot description, URDF)
Before this commit: robot tinykart, 10 links, 9 joints
Links:
- link laser_link: geometry collision cylinder length=0.01 radius=0.00762; visual cylinder length=0.01 radius=0.00762
Joints:
- joint laser_to_base_link: origin xyz=0.2722 0 0.3556 rpy=0 0 0 -> xyz=-0.2722 0 0.2 rpy=0 0 0

Commit message: fix urdf and nav

File: tinykart_description/urdf/tinykart.urdf (robot description, URDF)
Before this commit: robot tinykart, 10 links, 9 joints
Links:
- link base_link: mass 2 -> 1
- link left_front_wheel_rack: mass 1.125 -> 0.001
- link right_front_wheel: mass 1.125 -> 0.1
- link right_front_wheel_rack: mass 1.125 -> 0.001

File: tinykart_description/urdf/tinykart_robot.urdf (robot description, URDF)
Before this commit: robot tinykart, 10 links, 9 joints
Links:
- link imu_link: mass 1 -> 0
- link left_front_wheel_rack: mass 1.125 -> 0.001
- link right_front_wheel: mass 1.125 -> 0.1
- link right_front_wheel_rack: mass 1.125 -> 0.001
Joints:
- joint imu_link_to_base_link: origin xyz=-0.012 0 0.5588 rpy=0 0 0 -> xyz=-0.012 0 0.3 rpy=0 0 0
- joint laser_to_base_link: origin xyz=-0.2722 0 0.2 rpy=0 0 0 -> xyz=0.2722 0 0.2 rpy=0 0 0

Commit message: Fix sim (#3)
* wip

* fix urdf and nav

File: tinykart_description/urdf/tinykart.urdf (robot description, URDF)
Before this commit: robot tinykart, 10 links, 9 joints
Links:
- link imu_link: mass 1 -> 0
- link laser_link: geometry collision cylinder length=0.01 radius=0.00762; visual cylinder length=0.01 radius=0.00762
- link left_front_wheel_rack: mass 1.125 -> 0.001
- link right_front_wheel: mass 1.125 -> 0.1
- link right_front_wheel_rack: mass 1.125 -> 0.001
Joints:
- joint imu_link_to_base_link: origin xyz=-0.012 0 0.5588 rpy=0 0 0 -> xyz=-0.012 0 0.3 rpy=0 0 0
- joint laser_to_base_link: origin xyz=0.2722 0 0.3556 rpy=0 0 0 -> xyz=0.2722 0 0.2 rpy=0 0 0

File: tinykart_description/urdf/tinykart_robot.urdf (robot description, URDF)
Before this commit: robot tinykart, 10 links, 9 joints
Links:
- link imu_link: mass 1 -> 0
- link laser_link: geometry collision cylinder length=0.01 radius=0.00762; visual cylinder length=0.01 radius=0.00762
- link left_front_wheel_rack: mass 1.125 -> 0.001
- link right_front_wheel: mass 1.125 -> 0.1
- link right_front_wheel_rack: mass 1.125 -> 0.001
Joints:
- joint imu_link_to_base_link: origin xyz=-0.012 0 0.5588 rpy=0 0 0 -> xyz=-0.012 0 0.3 rpy=0 0 0
- joint laser_to_base_link: origin xyz=0.2722 0 0.3556 rpy=0 0 0 -> xyz=0.2722 0 0.2 rpy=0 0 0
